File: hardware/m360-act/M360-ACT.kicad_pcb (KiCad board)
At the start: 2 copper layers, 0 parts

Commit message: feat(hardware): posicionamento da M360-ACT
Placa de 100 x 80 mm com os 26 componentes posicionados e 4 furos M3. Aqui o contorno não é
apertado como o da LP: a placa é parafusada na chapa perfurada do quadro, onde há espaço de
sobra, então os blocos ficaram folgados e os conectores todos em borda.

- alto à esquerda: Pro Mini deitado, com o header FTDI apontando para fora da borda, de modo
  que o adaptador entra sem esbarrar em nada;
- alto à direita: mezanino, com o SMA atravessando a borda direita (a antena fica dentro do
  quadro, conforme §5.2);
- meio: 74HCT244 e CD74HC4067, cada um com o seu desacoplamento;
- coluna da esquerda: borne de 5 V na borda, AMS1117 e capacitores;
- borda de baixo: os três RJ45 com a boca para fora e os cinco TVS logo atrás deles, antes de
  qualquer outra peça;
- borda direita: reed (o ímã é aproximado pela parede do quadro) e o divisor da vazão.

O furo H2 não ficou no canto: ali cairia embaixo do mezanino e obrigaria a parafusar a placa
antes de encaixar o módulo. Desceu para a faixa livre entre o mezanino e o reed.

DRC sem sobreposição de courtyard e sem erro de isolamento. Os 14 avisos são de serigrafia:
13 são as frentes dos conectores rente à borda (propositais, é por onde entram os plugues e o
fio do barramento) e 1 é o texto de referência do U1 sobre uma ilha do C3, que fica para o
acerto de serigrafia. As 104 ligações pendentes são o roteamento, ainda por fazer.

Pendência mecânica: os furos M3 estão nos cantos; conferir contra a malha de furos da chapa
perfurada do quadro antes de fabricar.

Co-Authored-By: Claude Opus 5 (1M context) <noreply@anthropic.com>
Claude-Session: https://claude.ai/code/session_01G3CpSsqAsoKgMUYE5MhRV7
Parts:
- added A1: Pro Mini 3V3 8MHz, M360:Arduino_ProMini_DeeKRobot, F.Cu at (115.0, 126.0)
- added C1: 10uF, Capacitor_SMD:C_0805_2012Metric, F.Cu at (112.0, 138.0)
- added C2: 100nF, Capacitor_SMD:C_0603_1608Metric, F.Cu at (112.0, 142.0)
- added C3: 10uF, Capacitor_SMD:C_0805_2012Metric, F.Cu at (106.0, 132.0)
- added C4: 100nF, Capacitor_SMD:C_0603_1608Metric, F.Cu at (112.0, 132.0)
- added C5: 100nF, Capacitor_SMD:C_0603_1608Metric, F.Cu at (135.0, 132.0)
- added C6: 100nF, Capacitor_SMD:C_0603_1608Metric, F.Cu at (165.0, 132.0)
- added C7: 1nF, Capacitor_SMD:C_0603_1608Metric, F.Cu at (182.0, 161.0)
- added H1: MountingHole_3.2mm_M3, MountingHole_3.2mm_M3, F.Cu at (104.0, 104.0)
- added H2: MountingHole_3.2mm_M3, MountingHole_3.2mm_M3, F.Cu at (196.0, 131.0)
- added H3: MountingHole_3.2mm_M3, MountingHole_3.2mm_M3, F.Cu at (104.0, 176.0)
- added H4: MountingHole_3.2mm_M3, MountingHole_3.2mm_M3, F.Cu at (196.0, 176.0)
- added J1: 5V do quadro, M360:TerminalBlock_WJ500V-5.08-2P, F.Cu at (106.0, 150.0)
- added J2: M360-RF, M360:M360-RF_Soquete_2x05, F.Cu at (172.8, 108.4)
- added J3: RJ45 RELES-A, M360:RJ45_R-RJ45R08P-A004, F.Cu at (120.0, 171.3)
- added J4: RJ45 RELES-B, M360:RJ45_R-RJ45R08P-A004, F.Cu at (140.0, 171.3)
- added J5: RJ45 SENSORES, M360:RJ45_R-RJ45R08P-A004, F.Cu at (160.0, 171.3)
- added R1: 10k, Resistor_SMD:R_0603_1608Metric, F.Cu at (150.0, 112.0)
- added R2: 10k, Resistor_SMD:R_0603_1608Metric, F.Cu at (150.0, 120.0)
- added R3: 10k, Resistor_SMD:R_0603_1608Metric, F.Cu at (176.0, 158.0)
- added R4: 20k, Resistor_SMD:R_0603_1608Metric, F.Cu at (176.0, 164.0)
- added SW1: Reed, M360:Reed_Littelfuse_59170, F.Cu at (190.0, 145.0)
- added U1: AMS1117-3.3, Package_TO_SOT_SMD:SOT-223-3_TabPin2, F.Cu at (106.0, 138.0)
- added U2: 74HCT244, Package_SO:SOIC-20W_7.5x12.8mm_P1.27mm, F.Cu at (125.0, 140.0)
- added U3: CD74HC4067, Package_SO:SOIC-24W_7.5x15.4mm_P1.27mm, F.Cu at (155.0, 140.0)
- added U4: SRV05-4, Package_TO_SOT_SMD:SOT-23-6, F.Cu at (115.0, 160.5)
- added U5: SRV05-4, Package_TO_SOT_SMD:SOT-23-6, F.Cu at (127.0, 160.5)
- added U6: SRV05-4, Package_TO_SOT_SMD:SOT-23-6, F.Cu at (139.0, 160.5)
- added U7: SRV05-4, Package_TO_SOT_SMD:SOT-23-6, F.Cu at (151.0, 160.5)
- added U8: SRV05-4, Package_TO_SOT_SMD:SOT-23-6, F.Cu at (163.0, 160.5)
Other:
- board outline added: 100 x 80 mm

Commit message: feat(hardware): roteamento, planos de terra e serigrafia da M360-ACT
Regras da placa antes de rotear: isolamento 0,2 mm, trilha 0,25 mm e via 0,6/0,3 mm (as
padrão vinham com isolamento 0).

Roteamento pelo Freerouting 1.9.0 chamado direto na linha de comando, como na LP — o
autoroute do MCP exige Java 21 ou Docker, e aqui há Java 17, que basta para a versão 1.9.
Fluxo: export DSN pelo MCP, `java -jar freerouting.jar -de ... -do ... -mp 20`, import SES
pelo MCP. Resultado: **463 trilhas e 23 vias, zero ligações pendentes** (eram 104) e nenhum
erro de isolamento. O roteador emitiu dois avisos internos (`CalcFromSide: start corner was
not found`) que não tiveram consequência — quem atestou isso foi o DRC, não o log.

Planos de terra nas duas faces, isolamento de 0,25 mm, preenchidos com
`kicad-cli pcb drc --refill-zones --save-board` (o refill_zones do MCP arrisca falha de
segmentação).

O preenchimento expôs um erro de haste térmica insuficiente no pino 8 do J3, o pad de terra
do RJ45 — o mesmo caso já visto na LP, com o mesmo footprint e o mesmo campo de pinos
escalonado de 1,02 mm. Duas correções:

- hastes de 0,35 mm com folga de 0,3 mm (eram 0,5/0,5) nas duas zonas: cabem no anel apertado
  dos pads THT e preservam o alívio térmico, que é o que torna a solda manual viável;
- ligação sólida no pino 8 do J3, onde nem a haste fina cabe. É o pad de terra do chicote:
  ligação sólida dá o melhor retorno de massa, ao custo de mais calor na solda desse pad.

Serigrafia: o texto de referência do U1 saiu de cima da ilha 2 do C3 e foi para a faixa livre
entre o corpo do regulador e o borne J1. Acrescentado "Viridiotech.com.br" na área vazia
entre o CD74HC4067 e o reed.

Continuam apenas os avisos de serigrafia das frentes dos conectores rente à borda — três RJ45
e o borne de 5 V —, propositais: é por onde entram os plugues e o fio do barramento.

Verificação: a presença das trilhas e das zonas foi conferida no arquivo em disco a cada
etapa, e não pelo retorno do MCP, que r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
Routing:
- net GND: track 0.00 -> 432.9 mm, vias 0 -> 1
- net +5V: track 0.00 -> 226.8 mm
- net 3V3: track 0.00 -> 95.6 mm
- net FLOW_DIV: track 0.00 -> 91.2 mm
- net REED: track 0.00 -> 79.9 mm
- net REL_NFT: track 0.00 -> 76.3 mm, vias 0 -> 1
- net DIO0: track 0.00 -> 73.8 mm
- net AUX_A6: track 0.00 -> 70.4 mm, vias 0 -> 1
- net REL_CH2: track 0.00 -> 68.0 mm, vias 0 -> 1
- net REL_CH3: track 0.00 -> 65.7 mm, vias 0 -> 1
- net REL_CH6: track 0.00 -> 59.7 mm
- net REL_CH0: track 0.00 -> 57.8 mm, vias 0 -> 1
- net OE_N: track 0.00 -> 57.2 mm, vias 0 -> 2
- net REL_CH5: track 0.00 -> 56.7 mm, vias 0 -> 2
- net NSS: track 0.00 -> 55.5 mm
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- added copper zone on B.Cu, net GND
- added copper zone on F.Cu, net GND
Other:
- board text added: "Viridiotech.com.br"
