File: hardware/m360-gw/M360-GW.kicad_sch (KiCad schematic)
At the start: 15 parts, among them J1 Mezanino M360-RF, J2 5 V ext, SW1 AP / reset, U1 WEMOS D1 mini

Commit message: feat(hardware): posicionamento da M360-GW e LEDs fora da placa (J3)
Placa de 80 × 60 mm, 17 footprints (12 peças, 4 furos M3 e o conector), DRC 0 violações.

Duas restrições comandaram o arranjo, e nenhuma das duas aparece no DRC:

- o mezanino M360-RF ocupa 34,2 × 23 mm **acima** do soquete, mas o courtyard do soquete tem só
  6,2 × 13,8 — confiar nele teria colocado peças embaixo do módulo. J1 fica em x = borda − 27,2
  para o SMA sair pela lateral, e conferi por número que a faixa x 145,8-180 / y 100-123 está
  vazia;
- o D1 mini traz keep-out sobre a antena, na mesma ponta onde fica o USB. Essa ponta encosta na
  borda de cima: a antena não irradia para dentro do cobre e o cabo entra sem abrir a caixa.

Pelo mesmo motivo o H2 não fica no canto — ali cairia sob o mezanino, e a placa teria de ser
parafusada antes de encaixar o módulo. Mesma armadilha já evitada na ACT.

Os LEDs saíram da placa: ficam no painel da caixa e o J3 (JST XH) leva os três pares ao chicote.
São **6 vias em pares ânodo/cátodo**, e não 4 com terra comum, porque o verde é ativo em LOW — o
cátodo dele vai ao D4, não ao GND, de modo que não existe terra comum aos três. Com pares
dedicados os três são ligados da mesma forma no chicote apesar dessa assimetria, e o XH é
chaveado, o que impede inversão no campo. Os resistores de 1 kΩ ficam a bordo: limitação de
corrente não deve viajar no cabo.

O primeiro DRC acusou 5 violações, quatro delas com uma causa só: **girado 90°, o resistor não
fica centrado na origem** — o courtyard vai de y − 11,25 a y + 1,10, quase todo acima do ponto
informado. A fileira subia até 131,75 e entrava no U1, que termina em 134,79. O cálculo ficou
registrado como comentário no place_gw.py, porque se repete na próxima placa. A quinta violação
era o texto de referência do H1 cortado pela borda; como os furos são board-only e ficam fora da
BOM e do arquivo de posição, a serigrafia deles passou a invisível.

Verificação: a troca dos LEDs pelo conector alterou a netlist exatam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
Parts:
- removed D1: vermelho, LED_THT:LED_D3.0mm, symbol Device:LED
- removed D2: amarelo, LED_THT:LED_D3.0mm, symbol Device:LED
- removed D3: verde, LED_THT:LED_D3.0mm, symbol Device:LED
- added J3: LEDs (painel), Connector_JST:JST_XH_B6B-XH-A_1x06_P2.50mm_Vertical, symbol Connector_Generic:Conn_01x06
Connections:
- net GND: now also J3.2 (Pin_2), J3.4 (Pin_4)
- net LED_GREEN_A: now also J3.5 (Pin_5)
- net LED_GREEN_K: now also J3.6 (Pin_6)
- net LED_RED_A: now also J3.1 (Pin_1)
- net LED_YELLOW_A: now also J3.3 (Pin_3)

Commit message: feat(hardware): LP e ACT rerroteadas com o botão; GND volta a ser roteado
Conclui a troca do reed pelo botão iniciada em 0948368, que parou no esquemático.

Placas, para cada uma: del_fp.py SW1 → sincronização com o esquemático → place_*.py →
clear_tracks.py → export_dsn → dsn_sem_plano.py → Freerouting → import_ses →
zone_thermals.py → DRC com refill.

- M360-LP: 572 trilhas, 44 vias. DRC com 0 erros e 0 desconectados; restam os 8
  silk_edge_clearance dos RJ45, que já existiam.
- M360-ACT: 489 trilhas, 24 vias. DRC com 0 erros e 0 desconectados; restam os 13
  silk_edge_clearance, que já existiam. J1 em rot 0, como o place_act.py já pedia.
- Redes de todos os pads conferidas contra o HEAD: só o SW1 mudou. Trilhas todas de 0,25 mm.
- Paridade esquemático × placa com as mesmas contagens da base (237 e 195); some o
  footprint_symbol_mismatch do SW1.

**O GND não era roteado — e era isso que partia o plano.** Com zona de GND na placa, o DSN
declara `plane GND` e o Freerouting não desenha um fio de terra sequer. O primeiro roteamento
(bf701dc, 88 segmentos de GND) foi feito antes de as zonas existirem; todo rerroteamento
posterior perdia esse terra. Rerroteada com o DSN como sai do KiCad, a LP deu 16
unconnected_items, todos "Zona [GND]"; tirando as declarações plane, 0 — 100 segmentos de GND
na LP e 95 na ACT. Explica também os 15 desconectados imóveis da sessão anterior (§11.6).
Novo `tools/dsn_sem_plano.py`, e a §11 corrigida: 11.2, 11.4, 11.5 e 11.6.

Ajustes que o DRC pediu depois do rerroteamento:
- J4 da ACT, pino 8: starved_thermal → ligação sólida (pad_zone_connect.py), como o J3;
- silk_lp.py: referência do SW1 saía sobre "M360-LP"; vai para (172, 155);
- silk_act.py: referência do U1 encostava no J1, agora em rot 0; sobe para y = 143.

Botão: SHOU HAN TS665CJ, C393938, tátil 6 × 6 mm THT, SW1 nas três placas (LP, ACT e GW),
**solda manual e fora do PCBA**. Propriedade LCSC gravada nos três esquemáticos, com netlists
idênticas antes e depois. `add_lcsc.py` g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
Parts:
- SW1: LCSC (none) -> C393938
Changed lines of the file:
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@@
+			)
+		)
+		(property "LCSC" "C393938"
+			(at 107.95 157.48 0)
+			(hide yes)
+			(effects
+				(font
+					(size 1.27 1.27)
+				)
 			)
 		)

Commit message: feat(hardware): peças de solda manual fora do BOM e da posição; C13 da LP corrigido
Novo `tools/solda_manual.py`: marca as duas pontas pela referência — `in_bom no` e
`in_pos_files no` no símbolo, `exclude_from_bom` e `exclude_from_pos_files` no footprint. O BOM
sai do esquemático e a posição sai da placa; marcar um lado só faria a paridade divergir.

Aplicado:
- LP: SW1, J1, J2, A1, J4
- ACT: SW1, J3, J4, J5, A1, J2
- GW: SW1, J1

Conferido exportando BOM e posição antes e depois: saíram exatamente essas peças. Netlists
idênticas nas três; DRC e paridade com as mesmas contagens da base (LP 237, ACT 195, GW 69).
A propriedade LCSC fica nos símbolos, para a compra (§9.1).

**Defeito corrigido:** o C13 da LP (100 nF 0603) carregava o código do reed, C315909, desde
bc651ca — a JLCPCB montaria um reed no lugar do capacitor. Agora C14663, como os demais 100 nF,
pelo `add_lcsc.py --set`.

Também na §9.1: espaçamento de 6,5 × 4,5 mm do TS665CJ confirmado contra o datasheet.

Registrado na §9, sem correção: a ACT e a GW não têm código LCSC em peça nenhuma, e os
PWR_FLAG da GW saem no BOM. Bornes (J1 da ACT, J2 da GW) e JST (J3 da LP e da GW) continuam no
BOM, por não estarem na lista desta decisão.

Co-Authored-By: Claude Opus 5 (1M context) <noreply@anthropic.com>
Claude-Session: https://claude.ai/code/session_012t7RkcrXvvpDVjKVimNu18
Parts:
- J1, SW1: now left out of the parts list
Changed lines of the file:
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@@
 		(body_style 1)
 		(exclude_from_sim no)
-		(in_bom yes)
-		(on_board yes)
-		(in_pos_files yes)
+		(in_bom no)
+		(on_board yes)
+		(in_pos_files no)
 		(dnp no)
 		(property "Reference" "J1"
@@
 		(body_style 1)
 		(exclude_from_sim no)
-		(in_bom yes)
-		(on_board yes)
-		(in_pos_files yes)
+		(in_bom no)
+		(on_board yes)
+		(in_pos_files no)
 		(dnp no)
 		(property "Reference" "SW1"

Commit message: feat(hardware): códigos LCSC na M360-ACT e na M360-GW
Até aqui só a LP tinha código: o `add_lcsc.py` conhece apenas o mapa dela. Gravados com
`add_lcsc.py --set`, cada código conferido no catálogo local (estoque, encapsulamento, tipo).
Netlists idênticas antes e depois nas duas placas.

ACT — todas as peças, menos o Pro Mini (como na LP):
- C1, C3 10 µF 0805 C15850 · C2, C4–C6 100 nF C14663 · C7 1 nF C1588 — basic
- R1–R3 10 kΩ C25804 · R4 20 kΩ C4184 — basic
- U1 AMS1117-3.3 C6186 (basic) · U2 74HCT244 C5978 · U3 CD74HC4067 C496123 · U4–U8 SRV05-4 C558418
- J1 borne C8465 · J2 soquete C492399 · J3–J5 RJ45 C385834

GW — toda THT, sem nenhuma basic:
- C1 10 µF eletrolítico D5 P2 C106654 · C2–C4 100 nF C84772
- R1–R3 1 kΩ C57435 · R4 10 kΩ C57436 (UNI-ROYAL, axial 1/4 W 1 %)
- J1 soquete C492399 · J2 borne C8465 · J3 JST B6B-XH-A C144397
- U1 D1 mini sem código: não existe no catálogo.

O 100 nF da GW é MLCC X7R com terminais, não disco: os discos em estoque são Y5V, que perdem
boa parte da capacitância com tensão e temperatura.

Atenção: o C25804 (10 kΩ) não está no catálogo de peças em estoque, e não há outro 10 kΩ 0603
basic — a alternativa é extended (C2906982). Afeta 11 posições da LP e 3 da ACT; registrado na
§9 para confirmar no site antes do pedido. §9.1 ganha as peças novas.

Co-Authored-By: Claude Opus 5 (1M context) <noreply@anthropic.com>
Claude-Session: https://claude.ai/code/session_012t7RkcrXvvpDVjKVimNu18
Parts:
- C1: LCSC (none) -> C106654
- C2, C3, C4: LCSC (none) -> C84772
- J1: LCSC (none) -> C492399
- J2: LCSC (none) -> C8465
- J3: LCSC (none) -> C144397
- R1, R2, R3: LCSC (none) -> C57435
- R4: LCSC (none) -> C57436
Changed lines of the file:
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@@
+			)
+		)
+		(property "LCSC" "C492399"
+			(at 175.26 110.49 0)
+			(hide yes)
+			(effects
+				(font
+					(size 1.27 1.27)
+				)
 			)
 		)
@@
 			)
 		)
+		(property "LCSC" "C8465"
+			(at 39.37 69.85 0)
+			(hide yes)
+			(effects
+				(font
+					(size 1.27 1.27)
+				)
+			)
+		)
 		(property "Datasheet" ""
 			(at 39.37 69.85 0)
@@
 			)
 		)
+		(property "LCSC" "C144397"
+			(at 95.25 175.26 0)
+			(hide yes)
+			(effects
+				(font
+					(size 1.27 1.27)
+				)
+			)
+		)
 		(property "Datasheet" ""
 			(at 95.25 175.26 0)
@@
 			)
 		)
+		(property "LCSC" "C84772"
+			(at 59.69 69.85 0)
+			(hide yes)
+			(effects
+				(font
+					(size 1.27 1.27)
+				)
+			)
+		)
 		(property "Datasheet" ""
 			(at 59.69 69.85 0)
@@
 			)
 		)
+		(property "LCSC" "C106654"
+			(at 74.93 91.44 0)
+			(hide yes)
+			(effects
+				(font
+					(size 1.27 1.27)
+				)
+			)
+		)
 		(property "Datasheet" ""
 			(at 74.93 91.44 0)
@@
 			)
 		)
+		(property "LCSC" "C84772"
+			(at 90.17 91.44 0)
+			(hide yes)
+			(effects
+				(font
+					(size 1.27 1.27)
+				)
+			)
+		)
 		(property "Datasheet" ""
 			(at 90.17 91.44 0)
@@
 			)
 		)
+		(property "LCSC" "C57435"
+			(at 39.37 134.62 0)
+			(hide yes)
+			(effects
+				(font
+					(size 1.27 1.27)
+				)
+			)
+		)
 		(property "Datasheet" ""
 			(at 39.37 134.62 0)
@@
 			)
 		)
+		(property "LCSC" "C57435"
+			(at 39.37 154.94 0)
+			(hide yes)
+			(effects
+				(font
+					(size 1.27 1.27)
+				)
+			)
+		)
 		(property "Datasheet" ""
 			(at 39.37 154.94 0)
@@
 			)
 		)
+		(property "LCSC" "C57435"
+			(at 39.37 175.26 0)
+			(hide yes)
+			(effects
+				(font
+					(size 1.27 1.27)
+				)
+			)
+		)
 		(property "Datasheet" ""
 			(at 39.37 175.26 0)
@@
 			)
 		)
+		(property "LCSC" "C57436"
+			(at 139.7 148.59 0)
+			(hide yes)
+			(effects
+				(font
+					(size 1.27 1.27)
+				)
+			)
+		)
 		(property "Datasheet" ""
 			(at 139.7 148.59 0)
@@
 			(effects
 				(font
+					(size 1.27 1.27)
+				)
+			)
+		)
+		(property "LCSC" "C84772"
+			(at 157.48 148.59 0)
+			(hide yes)
+			(effects
+				(font

Commit message: feat(hardware): esquemáticos corrigidos após análise adversarial; reed nas três placas; GW em SMD
⚠️ **Só esquemáticos.** Os três .kicad_pcb estão defasados e serão refeitos depois de uma nova
análise adversarial, até zerar os achados (pedido do usuário). ARQUITETURA §9 registra.

Correções da revisão (Fable 5.1, 2026-09-13):
- ACT #1: A6 da J5 com divisor 10 k (R5) / 20 k (R6) + 100 nF (C8); J5.3 e U8.3 vão para AUX_A6_IN.
  Antes, 5 V do par marrom chegavam direto ao ADC6 de um ATmega a 3,3 V.
- ACT #2: pull-up do /OE (R2) de +5V para 3V3 — A5 em alta impedância ficava a ~3,8 V.
- ACT #4: 7× 100 kΩ — pull-down em MUX_S0..S3, pull-up para 5 V em MUX_SIG/REL_NFT/REL_OXI.
- ACT #6: AMS1117 → ME6211C33M5 (C82942), estável com cerâmico.
- ACT #12: AO3401A (Q1) contra inversão no borne; J1.1 vai para VIN_RAW.
- GW #5/#12: Schottky SS14 (D1, C2480) em série de J2.1 (VIN_RAW) para +5V.
- Achados 3, 7, 8, 9, 10 e 11: documentação e regras de firmware (módulo TP4056 com DW01+8205;
  vazão com INPUT; calibração e analogReference do A6 da LP; chave do mezanino cortando o pino 10;
  FTDI sem VCC; orçamento do 3,3 V da GW).

Decisões do usuário:
- Reed switch Littelfuse 59170 (C315909) de volta na LP e na ACT e **no lugar do botão AP/reset da
  GW**, pela PCBA. Símbolo trocado por texto (pinagem idêntica): netlists idênticas.
- GW em SMD pela JLCPCB: R 0603, C1 10 µF 0805 (`Device:C`), C2–C4 100 nF 0603, códigos basic.
  Solda manual só U1 (D1 mini), J1, J2, J3. Os PWR_FLAG saem do BOM.
- Solda manual marcada só nos esquemáticos (`solda_manual.py --so-esquematico`, e `--desfazer` no
  SW1): LP J3; ACT J1; GW U1, J1, J2, J3.

Verificado nas três: netdiff contra a base lista só as mudanças acima (LP idêntica); campos de
todos os componentes comparados; símbolos de biblioteca embutidos comparados com o HEAD; ERC 0;
BOM com código LCSC em todas as linhas (exceto módulos); desenho conferido em PDF.

Três armadilhas medidas no caminho (ARQUITETURA §12):
- `replace_schematic_component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
Parts:
- removed C1: 10u, Capacitor_THT:CP_Radial_D5.0mm_P2.00mm, symbol Device:C_Polarized
- added C1: 10uF, Capacitor_SMD:C_0805_2012Metric, symbol Device:C
- added D1: SS14, Diode_SMD:D_SMA, symbol Device:D_Schottky
- C2, C3, C4: value 100n -> 100nF; footprint Capacitor_THT:C_Disc_D5.0mm_W2.5mm_P5.00mm -> Capacitor_SMD:C_0603_1608Metric; LCSC C84772 -> C14663
- J2, J3, U1: now left out of the parts list
- R1, R2, R3: footprint Resistor_THT:R_Axial_DIN0207_L6.3mm_D2.5mm_P10.16mm_Horizontal -> Resistor_SMD:R_0603_1608Metric; LCSC C57435 -> C21190
- R4: footprint Resistor_THT:R_Axial_DIN0207_L6.3mm_D2.5mm_P10.16mm_Horizontal -> Resistor_SMD:R_0603_1608Metric; LCSC C57436 -> C25804
- SW1: value AP / reset -> Reed; footprint Button_Switch_THT:SW_PUSH_6mm -> M360:Reed_Littelfuse_59170; symbol Switch:SW_Push -> Switch:SW_Reed; LCSC C393938 -> C315909; now in the parts list
Connections:
- net +3V3: now also C1.1
- net +5V: now also D1.1 (K); no longer J2.1 (Pin_1)
- net GND: now also C1.2
- new net VIN_RAW: D1.2 (A), J2.1 (Pin_1)

Commit message: fix(hardware): esquemáticos — correções da 2ª análise adversarial
⚠️ Só esquemáticos; as placas continuam defasadas de propósito até zerar os achados.

- LP #1 (firmware + documento): a referência DEFAULT é o VCC, e abaixo de ~3,31 V de bateria o
  MCP1700 sai de regulação — o A6 devolve sempre "3,3 V". O firmware corrige pelo VCC medido no
  bandgap (`readADCInternal()` de M360Power.cpp): VBAT = 3 × ADC_A6 × VCC / 1023. §4.1 e §9.
- ACT #2: entrada da vazão refeita — R3 10 kΩ em série, D1 BAT54WS (C7502694) do D3 para o 3V3,
  R4 de 20 kΩ para 100 kΩ (pull-down, sem pulsos falsos com o sensor desligado). Serve às unidades
  push-pull e às de coletor aberto com pull-up interno, que no divisor antigo davam só 2,5 V.
- ACT #3: R14–R20 100 kΩ nas entradas do 74HCT244 — pull-down em MUX_S0..S3_3V3, pull-up para 3V3
  em MUX_SIG_3V3, NFT_3V3 e OXI_3V3. O /OE cobria as saídas, não as entradas.
- GW #4: Q1 2N7002 (C8545) — o GPIO2 (boot) só comanda o gate; o LED verde vai do 3,3 V ao dreno.
  Curto do chicote para o GND acende o LED em vez de travar o boot. Verde passa a ativo em HIGH,
  como os outros — some a inversão pendente no M360Leds.cpp.
- ACT #5: nota de projeto — o divisor do A6 carrega a fonte com 30 kΩ (§5.2, §7).
- Documento: `MY_RFM95_RST_PIN` (D8 na LP, A3 na ACT) na §9; saem a linha "DHT11 no atuador" da §9
  e o buck XL1509 da §9.1, inconsistentes com a §5.

Verificado: netdiff contra o commit anterior só com as redes previstas (LP idêntica; ACT 10, GW 3);
campos dos componentes existentes inalterados (fora o valor do R4); símbolos de biblioteca
existentes inalterados; ERC 0 nas três; BOM com código LCSC em todas as linhas; desenho conferido
em PDF.

Co-Authored-By: Claude Opus 5 (1M context) <noreply@anthropic.com>
Claude-Session: https://claude.ai/code/session_012t7RkcrXvvpDVjKVimNu18
Parts:
- added Q1: 2N7002, Package_TO_SOT_SMD:SOT-23, symbol Transistor_FET:2N7002
Connections:
- net GND: now also Q1.2 (S)
- net LED_GREEN_K: now also Q1.3 (D); no longer U1.11 (D4)
- new net LED_GREEN: Q1.1 (G), U1.11 (D4)
Changed lines of the file:
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@@
+	(wire
+		(pts
+			(xy 53.34 185.42) (xy 40.64 185.42)
+		)
+		(stroke
+			(width 0)
+			(type default)
+		)
+	)
 	(wire
 		(pts
@@
 	(wire
 		(pts
+			(xy 60.96 190.5) (xy 60.96 196.85)
+		)
+		(stroke
+			(width 0)
+			(type default)
+		)
+	)
+	(wire
+		(pts
 			(xy 170.18 113.03) (xy 163.83 113.03)
 		)
@@
 		(pts
 			(xy 35.56 134.62) (xy 25.4 134.62)
+		)
+		(stroke
+			(width 0)
+			(type default)
+		)
+	)
+	(wire
+		(pts
+			(xy 60.96 180.34) (xy 60.96 166.37)
 		)
 		(stroke
@@
 		)
 	)
-	(label "LED_GREEN_K"
+	(label "LED_GREEN"
 		(at 134.62 110.49 180)
 		(effects
@@
 		)
 	)
+	(label "LED_GREEN_K"
+		(at 60.96 166.37 270)
+		(effects
+			(font
+				(size 1.27 1.27)
+			)
+			(justify right bottom)
+		)
+	)
 	(label "A0_BTN"
 		(at 93.98 157.48 0)
@@
 	)
 	(label "GND"
+		(at 60.96 196.85 90)
+		(effects
+			(font
+				(size 1.27 1.27)
+			)
+			(justify left bottom)
+		)
+	)
+	(label "GND"
 		(at 157.48 158.75 90)
 		(effects
@@
 	(label "VIN_RAW"
 		(at 27.94 69.85 0)
+		(effects
+			(font
+				(size 1.27 1.27)
+			)
+			(justify left bottom)
+		)
+	)
+	(label "LED_GREEN"
+		(at 40.64 185.42 0)
 		(effects
 			(font
@@
 					(unit 1)
 				)
+			)
+		)
+	)
+	(symbol
+		(lib_id "Transistor_FET:2N7002")
+		(at 58.42 185.42 0)
+		(unit 1)
+		(body_style 1)
+		(exclude_from_sim no)
+		(in_bom yes)
+		(on_board yes)
+		(in_pos_files yes)
+		(dnp no)
+		(property "Reference" "Q1"
+			(at 66.04 184.15 0)
+			(show_name no)
+			(do_not_autoplace no)
+			(effects
+				(font
+					(size 1.27 1.27)
+				)
+				(justify left)
+			)
+		)
+		(property "Value" "2N7002"
+			(at 66.04 186.69 0)
+			(show_name no)
+			(do_not_autoplace no)
+			(effects
+				(font
+					(size 1.27 1.27)
+				)
+				(justify left)
+			)
+		)
+		(property "Footprint" "Package_TO_SOT_SMD:SOT-23"
+			(at 58.42 185.42 0)
+			(hide yes)
+			(show_name no)
+			(do_not_autoplace no)
+			(effects
+				(font
+					(size 1.27 1.27)
+					(italic yes)
+				)
+				(justify left)
+			)
+		)
+		(property "Datasheet" "https://www.onsemi.com/pub/Collateral/NDS7002A-D.PDF"
+			(at 58.42 185.42 0)
+			(hide yes)
+			(show_name no)
+			(do_not_autoplace no)
+			(effects
+				(font
+					(size 1.27 1.27)
+				)
+				(justify left)
+			)
+		)
+		(property "Description" "0.115A Id, 60V Vds, N-Channel MOSFET, SOT-23"
+			(at 58.42 185.42 0)
+			(hide yes)
+			(show_name no)
+			(do_not_autoplace no)
+			(effects
+				(font
+					(size 1.27 1.27)
+				)
+			)
+		)
+		(property "LCSC" "C8545"
+			(at 58.42 185.42 0)
+			(hide yes)
+			(show_name no)
+			(do_not_autoplace no)
+			(effects
+				(font
+					(size 1.27 1.27)
+				)
+			)
+		)
+		(pin "1"
+		)
+		(pin "2"
+		)
+		(pin "3"
+		)
+		(instances
+			(project "M360-GW"
+				(path "/48a18d9a-df80-4072-896a-d7ca09082424"
+					(reference "Q1")
+					(unit 1)
+				)

Commit message: fix(hardware): esquemáticos — correções da 3ª análise adversarial
⚠️ Só esquemáticos; as placas continuam defasadas de propósito até zerar os achados.

- LP #1: 100 Ω em série (R26–R29, C22775) entre o TVS e o Pro Mini nas linhas de campo digitais.
  A1.18/19/25/26 passam às redes ONEWIRE_MCU, DHT_MCU, SDA_MCU e SCL_MCU; pull-ups e TVS ficam do
  lado do conector. O pino do ATmega deixa de dividir o surto com o TVS.
- ACT #2: 100 Ω em série (R21–R32) entre o CI e o TVS nas 12 linhas de relé — U3 I0–I9 em
  REL_CHx_MUX, U2 2Y1/2Y2 em REL_NFT_BUF/REL_OXI_BUF. Custa 0,2 V nos 2 mA do opto.
- ACT e GW #3: TVS SMAJ5.0A (D2, C2925443) do +5V ao GND, depois do Q1 (ACT) e do D1 (GW), contra
  DC-DC ajustável girado por engano. Símbolo `Device:D_Zener` — o `D_TVS` do KiCad é bidirecional.
- GW #4: nota — o LED azul do D1 mini no GPIO2 fica invertido em relação ao verde do painel.
- Regras: limiar de corte de TX ≥ 3,0 V por causa do BOD de 2,7 V (efuse 0xFD); confirmar os fuses
  dos clones DeeKRobot por ISP; `initLEDs` com argumentos trocados continua registrado. §9.

Verificado: netdiff contra o commit anterior só com as redes previstas (LP 8, ACT 26, GW 2);
campos dos componentes existentes inalterados; símbolos de biblioteca existentes inalterados
(entra só o D_Zener, sai o D_TVS); ERC 0; BOM com código LCSC em todas as linhas; desenho
conferido em PDF. O diff da LP é grande porque o arquivo passou pela primeira vez por
`kicad-cli sch upgrade --force` (§12).

No caminho: o MCP ignorou o ângulo pedido em `add_schematic_component` (todas as peças entraram em
rot 0) e, com as fileiras apertadas, os fios desenhados fundiram redes — o netdiff e o ERC pegaram,
e a geometria foi refeita antes do commit.

Co-Authored-By: Claude Opus 5 (1M context) <noreply@anthropic.com>
Claude-Session: https://claude.ai/code/session_012t7RkcrXvvpDVjKVimNu18
Parts:
- added D2: SMAJ5.0A, Diode_SMD:D_SMA, symbol Device:D_Zener
Connections:
- net +5V: now also D2.1 (K)
- net GND: now also D2.2 (A)
Changed lines of the file:
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@@
+	(wire
+		(pts
+			(xy 80.01 36.83) (xy 80.01 30.48)
+		)
+		(stroke
+			(width 0)
+			(type default)
+		)
+	)
 	(wire
 		(pts
@@
 		(pts
 			(xy 110.49 130.81) (xy 110.49 137.16)
+		)
+		(stroke
+			(width 0)
+			(type default)
+		)
+	)
+	(wire
+		(pts
+			(xy 80.01 44.45) (xy 80.01 50.8)
 		)
 		(stroke
@@
 		)
 	)
+	(label "+5V"
+		(at 80.01 50.8 90)
+		(effects
+			(font
+				(size 1.27 1.27)
+			)
+			(justify left bottom)
+		)
+	)
 	(label "GND"
 		(at 119.38 157.48 180)
@@
 			)
 			(justify left bottom)
+		)
+	)
+	(label "GND"
+		(at 80.01 30.48 270)
+		(effects
+			(font
+				(size 1.27 1.27)
+			)
+			(justify right bottom)
 		)
 	)
@@
 					(unit 1)
 				)
+			)
+		)
+	)
+	(symbol
+		(lib_id "Device:D_Zener")
+		(at 80.01 40.64 90)
+		(unit 1)
+		(body_style 1)
+		(exclude_from_sim no)
+		(in_bom yes)
+		(on_board yes)
+		(in_pos_files yes)
+		(dnp no)
+		(property "Reference" "D2"
+			(at 83.82 35.56 0)
+			(show_name no)
+			(do_not_autoplace no)
+			(effects
+				(font
+					(size 1.27 1.27)
+				)
+			)
+		)
+		(property "Value" "SMAJ5.0A"
+			(at 83.82 45.72 0)
+			(show_name no)
+			(do_not_autoplace no)
+			(effects
+				(font
+					(size 1.27 1.27)
+				)
+			)
+		)
+		(property "Footprint" "Diode_SMD:D_SMA"
+			(at 80.01 40.64 0)
+			(hide yes)
+			(show_name no)
+			(do_not_autoplace no)
+			(effects
+				(font
+					(size 1.27 1.27)
+				)
+			)
+		)
+		(property "LCSC" "C2925443"
+			(at 80.01 40.64 0)
+			(hide yes)
+			(effects
+				(font
+					(size 1.27 1.27)
+				)
+			)
+		)
+		(property "Datasheet" ""
+			(at 80.01 40.64 0)
+			(hide yes)
+			(show_name no)
+			(do_not_autoplace no)
+			(effects
+				(font
+					(size 1.27 1.27)
+				)
+			)
+		)
+		(property "Description" "TVS unidirecional (símbolo Zener: K no +5V)"
+			(at 80.01 40.64 0)
+			(hide yes)
+			(show_name no)
+			(do_not_autoplace no)
+			(effects
+				(font
+					(size 1.27 1.27)
+				)
+			)
+		)
+		(pin "1"
+		)
+		(pin "2"
+		)
+		(instances
+			(project "M360-GW"
+				(path "/48a18d9a-df80-4072-896a-d7ca09082424"
+					(reference "D2")
+					(unit 1)
+				)
