File: hardware/m360-gw/M360-GW.kicad_pcb (KiCad board)
At the start: 2 copper layers, 80 x 60 mm, 25 parts, among them J1 Mezanino M360-RF, J2 5 V ext, J3 LEDs (painel), Q1 2N7002, SW1 Reed, U1 WEMOS D1 mini

Commit message: feat(hardware): header 1x8 do nRF24 legado nas placas GW, LP e ACT
- esquemáticos: header 1x8 "nRF24 legado" (GW J4, LP J5, ACT J6; C492407,
  solda manual, fora do BOM e da posição) e 10 uF 0805 (C5/C16/C9, C15850)
  nas mesmas redes do soquete do mezanino: CE = DIO0, CSN = NSS, IRQ = DIO1
  (sem ligação na GW). Um rádio por placa: nRF24 OU mezanino RFM95W
- tools/add_nrf_header.py: grava símbolo, fios e labels por texto, embute o
  Conn_01x08 stock e confere colisão; netdiff só nas redes previstas, ERC 0,
  campos e lib_symbols inalterados nas três folhas
- placas rerroteadas sem apagar a fiação existente (DSN com fios fixos e
  cobertos por área proibida, mais áreas proibidas sobre os fiduciais);
  vias de GND junto do pino 8 e do capacitor; legenda "nRF24 OU mezanino"
  e "CE" no pino 1. GW 287 trilhas/43 vias, LP 855/135, ACT 939/141;
  DRC --severity-all 0/0, paridade idêntica, ordem_tvs 13/13 e 15/15
- fabricacao/ regerada: GW 15, LP 53, ACT 54 peças
- ARQUITETURA §2 (decisão 15), §4.2, §5.2, §6.1, §8, §9, §9.1; datasheet
  C492407 em docs/datasheets. Firmware pendente: MY_RF24_CE_PIN=5 (GW) e
  =2 (LP/ACT), a testar na bancada

Co-Authored-By: Claude Fable 5.1 <noreply@anthropic.com>
Claude-Session: https://claude.ai/code/session_01M8U92DFNnZt7SqLtzrKYSR
Parts:
- added C5: 10uF, Capacitor_SMD:C_0805_2012Metric, F.Cu at (163.0, 138.0)
- added J4: nRF24 legado, Connector_PinHeader_2.54mm:PinHeader_1x08_P2.54mm_Vertical, F.Cu at (149.7, 131.0)
Routing:
- net GND: track 213.9 -> 430.5 mm, vias 36 -> 38
- net +3V3: track 66.4 -> 100.5 mm, vias 2 -> 3
- net MISO: track 32.2 -> 59.9 mm
- net DIO0: track 52.4 -> 77.6 mm
- net MOSI: track 21.9 -> 45.8 mm
- net SCK: track 23.6 -> 43.9 mm
- net NSS: track 32.9 -> 48.9 mm
- net LED_GREEN: track 61.3 -> 53.3 mm
- net LED_RED: track 51.1 -> 52.0 mm
- net LED_GREEN_K: track 6.94 -> 7.69 mm
Other:
- board text added: "CE"
- board text added: "nRF24 OU mezanino"
