File: hardware/m360-rf/M360-RF.kicad_pcb (KiCad board)
At the start: 2 copper layers, 0 parts

Commit message: feat(hardware): layout da placa do mezanino M360-RF
Placa de 34,2 x 23 mm, 2 camadas, 1,6 mm. RFM95W no centro; header 2x5 na face de baixo, à esquerda; SMA Samtec na borda direita, alinhado ao pino ANA. Trilha de RF coplanar com terra (1,25 mm, gap 0,2 mm, ~5 mm). SPI reto até a coluna de dentro do header; DIO1, DIO0 e 3V3 contornam o rádio por cima, em F.Cu, sem cruzamentos. GND nas duas faces com 17 vias de costura, nenhuma sob o módulo. Referências de C1, C2 e J2 ocultas na serigrafia.

Pinagem do header reordenada para o layout (MISO/MOSI/SCK/NSS/RESET na coluna ímpar, DIO1/DIO0/3V3/GND/GND na par); esquemático religado e ERC sem violações. DRC do kicad-cli: 0 violações, 0 itens desconectados, 0 divergências com o esquemático. ARQUITETURA_FAMILIA.md: nova pinagem e interface mecânica do mezanino para os carriers.

Co-Authored-By: Claude Opus 5 (1M context) <noreply@anthropic.com>

Claude-Session: https://claude.ai/code/session_01G3CpSsqAsoKgMUYE5MhRV7
Parts:
- added C1: 100nF, Capacitor_SMD:C_0603_1608Metric, F.Cu at (130.2, 101.0)
- added C2: 22uF, Capacitor_SMD:C_0805_2012Metric, F.Cu at (132.2, 101.2)
- added J1: M360-RF 2x5, Connector_PinHeader_2.54mm:PinHeader_2x05_P2.54mm_Vertical, B.Cu at (107.5, 94.9)
- added J2: SMA borda, Connector_Coaxial:SMA_Samtec_SMA-J-P-H-ST-EM1_EdgeMount, F.Cu at (132.6, 107.0)
- added U1: RFM95W-915S2, RF_Module:HOPERF_RFM9XW_SMD, F.Cu at (120.0, 100.0)
Routing:
- net 3V3: track 0.00 -> 61.5 mm
- net DIO0: track 0.00 -> 46.5 mm
- net DIO1: track 0.00 -> 37.2 mm
- net GND: track 0.00 -> 8.85 mm, vias 0 -> 21
- net RESET: track 0.00 -> 5.39 mm
- net NSS: track 0.00 -> 5.21 mm
- net RF_ANT: track 0.00 -> 5.07 mm
- net SCK: track 0.00 -> 5.07 mm
- net MOSI: track 0.00 -> 5.00 mm
- net MISO: track 0.00 -> 4.98 mm
- added copper zone on B.Cu, net GND
- added copper zone on F.Cu, net GND
Other:
- board outline added: 34.2 x 23 mm
