File: hardware/m360-lp/M360-LP.kicad_pcb (KiCad board)
At the start: 2 copper layers, 86 x 62 mm, 64 parts, among them J1 RJ45 SOLO, J2 RJ45 CLIMA/AUX, J3 J_VIN 3,0-6V, J4 M360-RF, Q1 AO3401A, Q2 AO3401A, SW1 Reed, U1 MCP1700T-3302E/TT, U2 74HC4051, U3 SRV05-4, U4 SRV05-4, U5 SRV05-4

Commit message: feat(hardware): header 1x8 do nRF24 legado nas placas GW, LP e ACT
- esquemáticos: header 1x8 "nRF24 legado" (GW J4, LP J5, ACT J6; C492407,
  solda manual, fora do BOM e da posição) e 10 uF 0805 (C5/C16/C9, C15850)
  nas mesmas redes do soquete do mezanino: CE = DIO0, CSN = NSS, IRQ = DIO1
  (sem ligação na GW). Um rádio por placa: nRF24 OU mezanino RFM95W
- tools/add_nrf_header.py: grava símbolo, fios e labels por texto, embute o
  Conn_01x08 stock e confere colisão; netdiff só nas redes previstas, ERC 0,
  campos e lib_symbols inalterados nas três folhas
- placas rerroteadas sem apagar a fiação existente (DSN com fios fixos e
  cobertos por área proibida, mais áreas proibidas sobre os fiduciais);
  vias de GND junto do pino 8 e do capacitor; legenda "nRF24 OU mezanino"
  e "CE" no pino 1. GW 287 trilhas/43 vias, LP 855/135, ACT 939/141;
  DRC --severity-all 0/0, paridade idêntica, ordem_tvs 13/13 e 15/15
- fabricacao/ regerada: GW 15, LP 53, ACT 54 peças
- ARQUITETURA §2 (decisão 15), §4.2, §5.2, §6.1, §8, §9, §9.1; datasheet
  C492407 em docs/datasheets. Firmware pendente: MY_RF24_CE_PIN=5 (GW) e
  =2 (LP/ACT), a testar na bancada

Co-Authored-By: Claude Fable 5.1 <noreply@anthropic.com>
Claude-Session: https://claude.ai/code/session_01M8U92DFNnZt7SqLtzrKYSR
Parts:
- added C16: 10uF, Capacitor_SMD:C_0805_2012Metric, F.Cu at (169.0, 148.0)
- added J5: nRF24 legado, Connector_PinHeader_2.54mm:PinHeader_1x08_P2.54mm_Vertical, F.Cu at (147.1, 152.0)
Routing:
- net GND: track 297.0 -> 645.4 mm, vias 48 -> 52
- net MISO: track 26.9 -> 89.7 mm, vias 1 -> 2
- net SCK: track 36.8 -> 88.1 mm, vias 0 -> 1
- net MOSI: track 28.0 -> 77.6 mm, vias 0 -> 1
- net DIO0: track 43.3 -> 91.0 mm, vias 2 -> 6
- net 3V3: track 110.3 -> 155.6 mm
- net NSS: track 39.6 -> 81.3 mm
- net DIO1: track 22.5 -> 64.2 mm, vias 0 -> 2
- net SCL: track 50.3 -> 54.3 mm
- net VIN_RAW: track 41.3 -> 40.5 mm
- net ONEWIRE: track 35.8 -> 36.4 mm
- net SDA: track 59.3 -> 59.9 mm
- net SOIL4: track 26.2 -> 26.8 mm
- net SOIL6: track 39.4 -> 40.0 mm
- net VIN: track 64.5 -> 64.0 mm
Other:
- board text added: "CE"
- board text added: "nRF24 OU mezanino"
